File: pcb/Lower/Lower.kicad_sch (KiCad schematic)
At the start: 32 parts, among them J1 AudioJack3, J2 AudioJack3, J3 Barrel_Jack, J4 Conn_01x04, Q1 AO3401A, SW1 SW_Push_3PDT, U1 TL072

Commit message: [Lower] Fix LCSC part number for AO3401A (Was SOT-23-L3 instead of SOT-23)
Parts:
- Q1: LCSC C15127 -> C347476
Changed lines of the file:
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@@
       (effects (font (size 1.27 1.27)) hide)
     )
+    (pin "1")
+    (pin "2")
+    (pin "3")
     (pin "5")
     (pin "6")
     (pin "7")
+    (pin "4")
+    (pin "8")
   )
   (symbol (lib_id "Device:C") (at 220.345 92.71 0) (unit 1)
@@
       (effects (font (size 1.27 1.27)) (justify left) hide)
     )
-    (property "LCSC" "C15127" (id 4) (at 68.58 123.19 0)
+    (property "LCSC" "C347476" (id 4) (at 68.58 123.19 0)
       (effects (font (size 1.27 1.27)) hide)
     )
@@
     (pin "2")
     (pin "3")
+    (pin "5")
+    (pin "6")
+    (pin "7")
+    (pin "4")
+    (pin "8")
   )
   (symbol (lib_id "power:+9V") (at 210.185 76.2 0) (unit 1)
@@
       (effects (font (size 1.27 1.27)) hide)
     )
+    (pin "1")
+    (pin "2")
+    (pin "3")
+    (pin "5")
+    (pin "6")
+    (pin "7")
     (pin "4")
     (pin "8")
