File: pcb/Proto-Advanced/Proto-Advanced.kicad_sch (KiCad schematic)
At the start: 21 parts, among them J1 Conn_01x04, J10 Conn_01x01, J11 Conn_01x01, J12 Conn_01x01, J13 Conn_01x01, J14 Conn_01x01, J2 Conn_01x01, J3 Conn_01x01, J4 Conn_01x01, J41 Conn_01x01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

Commit message: [All] Add LCSC part number for JST connector
Parts:
- J1: value Conn_01x04 -> (none); footprint Connector_JST:JST_XH_B4B-XH-A_1x04_P2.50mm_Vertical -> (none); LCSC (none) -> C144395; now in the parts list
Changed lines of the file:
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@@
   )
   (symbol (lib_id "Connector_Generic:Conn_01x04") (at 48.26 29.21 0) (mirror x) (unit 1)
-    (in_bom no) (on_board yes)
+    (in_bom yes) (on_board yes)
     (property "Reference" "J1" (id 0) (at 51.435 29.2101 0)
       (effects (font (size 1.27 1.27)) (justify left))
     )
-    (property "Value" "Conn_01x04" (id 1) (at 44.45 21.59 0)
+    (property "Value" "" (id 1) (at 44.45 21.59 0)
       (effects (font (size 1.27 1.27)) (justify left))
     )
-    (property "Footprint" "Connector_JST:JST_XH_B4B-XH-A_1x04_P2.50mm_Vertical" (id 2) (at 48.26 29.21 0)
+    (property "Footprint" "" (id 2) (at 48.26 29.21 0)
       (effects (font (size 1.27 1.27)) hide)
     )
@@
       (effects (font (size 1.27 1.27)) hide)
     )
+    (property "LCSC" "C144395" (id 4) (at 48.26 29.21 0)
+      (effects (font (size 1.27 1.27)) hide)
+    )
