File: pcb/404_Frontpanel/404_Frontpanel.kicad_pcb (KiCad board)
At the start: 2 copper layers, 54.5 x 106.4 mm, 11 parts

Commit message: [404] Change my mind on the design. Wires it is.
Routing:
- net (no net): track 0.00 -> 281.9 mm, vias 0 -> 12
Changed lines of the file:
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@@
     (solder_mask_min_width 0.254)
     (aux_axis_origin 149.5 63.13)
-    (grid_origin 149.5 63.13)
+    (grid_origin 172.25 119.63)
     (pcbplotparams
       (layerselection 0x00010fc_ffffffff)
@@
     (effects (font (size 8 8) (thickness 1.2) italic))
   )
+  (segment (start 160.185 141.601) (end 163.868 137.918) (width 0.4) (layer "F.Cu") (net 0))
+  (segment (start 154.216 117.344) (end 153.073 117.344) (width 0.4) (layer "F.Cu") (net 0))
+  (segment (start 154.978 159.762) (end 154.978 162.81) (width 0.4) (layer "F.Cu") (net 0))
+  (segment (start 141.516 129.282) (end 135.42 135.378) (width 0.4) (layer "F.Cu") (net 0))
+  (segment (start 170.472 128.266) (end 174.79 128.266) (width 0.4) (layer "F.Cu") (net 0))
+  (segment (start 155.74 162.81) (end 155.74 159.254) (width 0.4) (layer "F.Cu") (net 0))
+  (segment (start 153.962 116.582) (end 152.692 116.582) (width 0.4) (layer "F.Cu") (net 0))
+  (segment (start 123.99 125.726) (end 128.054 125.726) (width 0.4) (layer "F.Cu") (net 0))
+  (segment (start 139.23 142.236) (end 139.738 142.236) (width 0.4) (layer "F.Cu") (net 0))
+  (segment (start 154.47 159.254) (end 154.978 159.762) (width 0.4) (layer "F.Cu") (net 0))
+  (segment (start 164.63 138.172) (end 158.534 144.268) (width 0.4) (layer "F.Cu") (net 0))
+  (segment (start 137.706 135.124) (end 137.706 137.41) (width 0.4) (layer "F.Cu") (net 0))
+  (segment (start 158.788 145.03) (end 165.392 138.426) (width 0.4) (layer "F.Cu") (net 0))
+  (segment (start 160.312 141.474) (end 160.312 138.172) (width 0.4) (layer "F.Cu") (net 0))
+  (segment (start 139.484 129.282) (end 131.864 136.902) (width 0.4) (layer "F.Cu") (net 0))
+  (segment (start 155.74 159.254) (end 155.232 158.746) (width 0.4) (layer "F.Cu") (net 0))
+  (segment (start 149.39 138.68) (end 150.66 137.41) (width 0.4) (layer "F.Cu") (net 0))
+  (segment (start 165.392 138.426) (end 165.392 136.394) (width 0.4) (layer "F.Cu") (net 0))
+  (segment (start 128.054 125.726) (end 132.88 120.9) (width 0.4) (layer "F.Cu") (net 0))
+  (segment (start 170.726 129.028) (end 164.63 135.124) (width 0.4) (layer "F.Cu") (net 0))
+  (segment (start 157.772 118.106) (end 160.312 120.646) (width 0.4) (layer "F.Cu") (net 0))
+  (segment (start 165.392 136.394) (end 166.154 135.632) (width 0.4) (layer "F.Cu") (net 0))
+  (segment (start 134.15 117.598) (end 136.944 114.804) (width 0.4) (layer "F.Cu") (net 0))
+  (segment (start 137.706 137.918) (end 139.484 139.696) (width 0.4) (layer "F.Cu") (net 0))
+  (segment (start 149.644 120.773) (end 149.644 121.154) (width 0.4) (layer "F.Cu") (net 0))
+  (segment (start 154.978 116.582) (end 154.216 117.344) (width 0.4) (layer "F.Cu") (net 0))
+  (segment (start 149.39 139.696) (end 149.39 138.68) (width 0.4) (layer "F.Cu") (net 0))
+  (segment (start 134.658 156.714) (end 132.88 158.492) (width 0.4) (layer "F.Cu") (net 0))
+  (segment (start 139.738 142.236) (end 141.008 143.506) (width 0.4) (layer "F.Cu") (net 0))
+  (segment (start 158.026 143.76) (end 160.185 141.601) (width 0.4) (layer "F.Cu") (net 0))
+  (segment (start 160.185 141.601) (end 160.312 141.474) (width 0.4) (layer "F.Cu") (net 0))
+  (segment (start 134.15 118.868) (end 134.15 117.598) (width 0.4) (layer "F.Cu") (net 0))
+  (segment (start 131.864 136.902) (end 131.864 145.538) (width 0.4) (layer "F.Cu") (net 0))
+  (segment (start 137.198 130.552) (end 138.468 129.282) (width 0.4) (layer "F.Cu") (net 0))
+  (segment (start 136.944 134.87) (end 136.944 137.41) (width 0.4) (layer "F.Cu") (net 0))
+  (segment (start 150.66 137.41) (end 153.454 137.41) (width 0.4) (layer "F.Cu") (net 0))
+  (segment (start 141.262 130.552) (end 136.944 134.87) (width 0.4) (layer "F.Cu") (net 0))
+  (segment (start 132.626 145.284) (end 133.388 146.046) (width 0.4) (layer "F.Cu") (net 0))
+  (segment (start 159.296 116.582) (end 154.978 116.582) (width 0.4) (layer "F.Cu") (net 0))
+  (segment (start 137.706 137.41) (end 137.706 137.918) (width 0.4) (layer "F.Cu") (net 0))
+  (segment (start 145.58 125.853) (end 145.072 126.361) (width 0.4) (layer "F.Cu") (net 0))
+  (segment (start 150.66 120.773) (end 153.327 118.106) (width 0.4) (layer "F.Cu") (net 0))
+  (segment (start 164.63 135.124) (end 164.63 138.172) (width 0.4) (layer "F.Cu") (net 0))
+  (segment (start 163.868 137.918) (end 163.868 134.87) (width 0.4) (layer "F.Cu") (net 0))
+  (segment (start 151.676 115.566) (end 151.676 114.804) (width 0.4) (layer "F.Cu") (net 0))
+  (segment (start 153.327 118.106) (end 157.772 118.106) (width 0.4) (layer "F.Cu") (net 0))
+  (segment (start 133.642 156.46) (end 127.292 162.81) (width 0.4) (layer "F.Cu") (net 0))
+  (segment (start 140.5 129.282) (end 132.626 137.156) (width 0.4) (layer "F.Cu") (net 0))
+  (segment (start 153.454 114.804) (end 144.31 123.948) (width 0.4) (layer "F.Cu") (net 0))
+  (segment (start 150.66 121.154) (end 150.66 120.773) (width 0.4) (layer "F.Cu") (net 0))
+  (segment (start 138.214 142.744) (end 140.246 144.776) (width 0.4) (layer "F.Cu") (net 0))
+  (segment (start 135.42 135.378) (end 135.42 138.934) (width 0.4) (layer "F.Cu") (net 0))
+  (segment (start 141.516 131.314) (end 137.706 135.124) (width 0.4) (layer "F.Cu") (net 0))
+  (segment (start 137.198 130.552) (end 130.34 130.552) (width 0.4) (layer "F.Cu") (net 0))
+  (segment (start 153.454 137.41) (end 154.216 136.648) (width 0.4) (layer "F.Cu") (net 0))
+  (segment (start 133.642 153.92) (end 133.642 156.46) (width 0.4) (layer "F.Cu") (net 0))
+  (segment (start 132.88 117.852) (end 135.928 114.804) (width 0.4) (layer "F.Cu") (net 0))
+  (segment (start 131.864 145.538) (end 132.626 146.3) (width 0.4) (layer "F.Cu") (net 0))
+  (segment (start 163.868 134.87) (end 170.472 128.266) (width 0.4) (layer "F.Cu") (net 0))
+  (segment (start 136.944 137.41) (end 136.944 141.474) (width 0.4) (layer "F.Cu") (net 0))
+  (segment (start 156.502 160.524) (end 157.01 161.032) (width 0.4) (layer "F.Cu") (net 0))
+  (segment (start 153.073 117.344) (end 149.644 120.773) (width 0.4) (layer "F.Cu") (net 0))
+  (segment (start 143.548 123.694) (end 151.676 115.566) (width 0.4) (layer "F.Cu") (net 0))
+  (segment (start 155.994 158.238) (end 156.502 158.746) (width 0.4) (layer "F.Cu") (net 0))
+  (segment (start 132.88 120.9) (end 132.88 117.852) (width 0.4) (layer "F.Cu") (net 0))
+  (segment (start 136.944 141.474) (end 138.214 142.744) (width 0.4) (layer "F.Cu") (net 0))
+  (segment (start 132.626 137.156) (end 132.626 145.284) (width 0.4) (layer "F.Cu") (net 0))
+  (segment (start 156.502 158.746) (end 156.502 160.524) (width 0.4) (layer "F.Cu") (net 0))
+  (segment (start 146.088 124.329) (end 144.818 125.599) (width 0.4) (layer "F.Cu") (net 0))
+  (segment (start 155.74 114.804) (end 153.962 116.582) (width 0.4) (layer "F.Cu") (net 0))
+  (segment (start 134.658 154.174) (end 134.658 156.714) (width 0.4) (layer "F.Cu") (net 0))
+  (segment (start 174.79 129.028) (end 170.726 129.028) (width 0.4) (layer "F.Cu") (net 0))
+  (segment (start 152.692 116.582) (end 144.818 124.456) (width 0.4) (layer "F.Cu") (net 0))
+  (via (at 160.312 138.172) (size 1) (drill 0.6) (layers "F.Cu" "B.Cu") (net 0))
+  (via (at 135.42 138.934) (size 1) (drill 0.6) (layers "F.Cu" "B.Cu") (net 0))
+  (via (at 160.312 120.646) (size 1) (drill 0.6) (layers "F.Cu" "B.Cu") (net 0))
+  (via (at 130.34 130.552) (size 1) (drill 0.6) (layers "F.Cu" "B.Cu") (net 0))
+  (via (at 134.15 118.868) (size 1) (drill 0.6) (layers "F.Cu" "B.Cu") (net 0))
+  (via (at 166.154 135.632) (size 1) (drill 0.6) (layers "F.Cu" "B.Cu") (net 0))
+  (via (at 159.296 116.582) (size 1) (drill 0.6) (layers "F.Cu" "B.Cu") (net 0))
+  (via (at 139.484 139.696) (size 1) (drill 0.6) (layers "F.Cu" "B.Cu") (net 0))
+  (via (at 157.01 161.032) (size 1) (drill 0.6) (layers "F.Cu" "B.Cu") (net 0))
+  (via (at 139.23 142.236) (size 1) (drill 0.6) (layers "F.Cu" "B.Cu") (net 0))
+  (via (at 132.88 158.492) (size 1) (drill 0.6) (layers "F.Cu" "B.Cu") (net 0))
+  (via (at 154.216 136.648) (size 1) (drill 0.6) (layers "F.Cu" "B.Cu") (net 0))
   (zone (net 0) (net_name "") (layers F&B.Cu) (hatch edge 0.508)
     (connect_pads (clearance 0.508))
