File: pcb/UpperRaw/UpperRaw.kicad_pcb (KiCad board)
At the start: 2 copper layers, 52 x 63 mm, 15 parts, among them J1 Conn_01x04

Commit message: [All] Flip board to board connector on upper PCB (obstructed some silk)
Parts:
- added C1: 22uF, Capacitor_SMD:C_1206_3216Metric, F.Cu at (63.1, 105.3)
- added C100: 100uF, Capacitor_THT:CP_Radial_D5.0mm_P2.00mm, F.Cu at (94.5, 92.6)
- added C101: 10uF, Capacitor_SMD:C_0805_2012Metric, F.Cu at (68.2, 105.2)
- added C102: 220nF, Capacitor_SMD:C_0603_1608Metric, F.Cu at (62.3, 108.3)
- added JP100: Jmp, Jumper:SolderJumper-2_P1.3mm_Open_TrianglePad1.0x1.5mm, F.Cu at (72.6, 105.4)
- added R1: 10K, Resistor_SMD:R_0603_1608Metric, F.Cu at (66.3, 108.3)
- added R100: 1M, Resistor_SMD:R_0603_1608Metric, F.Cu at (84.8, 104.9)
- added R101: 2M2, Resistor_SMD:R_0603_1608Metric, F.Cu at (100.8, 90.6)
- added R102: 390R, Resistor_SMD:R_0603_1608Metric, F.Cu at (94.2, 97.1)
- added R103: 2k2, Resistor_SMD:R_0603_1608Metric, F.Cu at (80.8, 107.4)
- added R2: 10K, Resistor_SMD:R_0603_1608Metric, F.Cu at (80.8, 104.9)
- added SW100: SW_DPDT_x2, MeineBib:Switch_toggle_DPDT_Print, F.Cu at (76.2, 82.2)
- added SW101: SW_DPDT_x2, MeineBib:Switch_toggle_DPDT_Print, F.Cu at (99.1, 82.2)
- added SW102: SW_SPDT, MeineBib:Switch_toggle_SPDT_Print, F.Cu at (64.8, 82.2)
- added SW103: SW_SPDT, MeineBib:Switch_toggle_SPDT_Print, F.Cu at (64.8, 96.5)
- added SW200: SW_DPDT_x2, MeineBib:Switch_toggle_DPDT_Print, F.Cu at (112.9, 82.2)
- added SW201: SW_DPDT_x2, MeineBib:Switch_toggle_DPDT_Print, F.Cu at (85.3, 96.5)
- added SW202: SW_SPDT, MeineBib:Switch_toggle_SPDT_Print, F.Cu at (87.7, 82.2)
- added SW203: SW_SPDT, MeineBib:Switch_toggle_SPDT_Print, F.Cu at (73.8, 96.5)
- added TP100: TP, TestPoint:TestPoint_Pad_D2.0mm, F.Cu at (76.8, 105.7)
- moved J1 7.57 mm to (153.2, 128.0), turned to 180 degrees
Connections:
- J1 pad 1: GND -> Upper_PCB_Input
- J1 pad 2: +9V -> Upper_PCB_Output
- J1 pad 3: Upper_PCB_Output -> +9V
- J1 pad 4: Upper_PCB_Input -> GND

Commit message: [404][UpperRaw] Apply learned lessons from TOP:
- Name on silk etc. is now a text variable
- Optimized copypasta parts
- Set pot footprint to my modified one
- Rename pots ro always be RV1-6
- Use text variables for pot names
- Show pot values on silk
- Update board constraints to JLCPCB capabilities
- Add Gndpour to UpperRaw
- Set "Not in schematic" for OSHW logo
Parts:
- removed C100: 100uF, Capacitor_THT:CP_Radial_D5.0mm_P2.00mm
- renumbered RV102 to RV1, RV101 to RV2, RV100 to RV3, RV202 to RV4, RV201 to RV5, RV200 to RV6
Routing:
- added copper zone on B.Cu, net GND
- added copper zone on F.Cu, net GND
Other:
- board text added: "${RV1}"
- board text added: "${RV2}"
- board text added: "${RV3}"
- board text added: "${RV4}"
- board text added: "${RV5}"
- board text added: "${RV6}"
- board text removed: "Base"
- board text removed: "Pot"
