File: pcb/UpperRaw/UpperRaw.kicad_sch (KiCad schematic)
At the start: 27 parts, among them J1 Conn_01x04, SW100 SW_DPDT_x2, SW101 SW_DPDT_x2, SW102 SW_SPDT, SW103 SW_SPDT, SW200 SW_DPDT_x2, SW201 SW_DPDT_x2, SW202 SW_SPDT, SW203 SW_SPDT

Commit message: [All] Flip board to board connector on upper PCB (obstructed some silk)
Parts:
- gave numbers to parts that had none: 3
Connections:
- net +9V: now also J1.3 (Pin_3); no longer J1.2 (Pin_2)
- net GND: now also J1.4 (Pin_4); no longer J1.1 (Pin_1)
- net Upper_PCB_Input: now also J1.1 (Pin_1); no longer J1.4 (Pin_4)
- net Upper_PCB_Output: now also J1.2 (Pin_2); no longer J1.3 (Pin_3)
Changed lines of the file:
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@@
   (symbol (lib_id "power:GND") (at 39.37 74.93 0) (unit 1)
     (in_bom yes) (on_board yes)
-    (property "Reference" "#PWR?" (id 0) (at 39.37 81.28 0)
+    (property "Reference" "#PWR0102" (id 0) (at 39.37 81.28 0)
       (effects (font (size 1.27 1.27)) hide)
     )
@@
   (symbol (lib_id "power:+9V") (at 29.21 52.07 0) (unit 1)
     (in_bom yes) (on_board yes)
-    (property "Reference" "#PWR?" (id 0) (at 29.21 55.88 0)
+    (property "Reference" "#PWR0104" (id 0) (at 29.21 55.88 0)
       (effects (font (size 1.27 1.27)) hide)
     )
@@
     (pin "6")
   )
-  (symbol (lib_id "Connector_Generic:Conn_01x04") (at 48.26 29.21 0) (mirror x) (unit 1)
-    (in_bom yes) (on_board yes)
-    (property "Reference" "J1" (id 0) (at 51.435 29.2101 0)
-      (effects (font (size 1.27 1.27)) (justify left))
-    )
-    (property "Value" "Conn_01x04" (id 1) (at 44.45 21.59 0)
-      (effects (font (size 1.27 1.27)) (justify left))
-    )
-    (property "Footprint" "Connector_JST:JST_XH_B4B-XH-A_1x04_P2.50mm_Vertical" (id 2) (at 48.26 29.21 0)
-      (effects (font (size 1.27 1.27)) hide)
-    )
-    (property "Datasheet" "~" (id 3) (at 48.26 29.21 0)
-      (effects (font (size 1.27 1.27)) hide)
-    )
-    (property "LCSC" "C144395" (id 4) (at 48.26 29.21 0)
+  (symbol (lib_id "Connector_Generic:Conn_01x04") (at 48.26 26.67 0) (unit 1)
+    (in_bom yes) (on_board yes)
+    (property "Reference" "J1" (id 0) (at 51.435 26.6699 0)
+      (effects (font (size 1.27 1.27)) (justify left))
+    )
+    (property "Value" "Conn_01x04" (id 1) (at 44.45 34.29 0)
+      (effects (font (size 1.27 1.27)) (justify left))
+    )
+    (property "Footprint" "Connector_JST:JST_XH_B4B-XH-A_1x04_P2.50mm_Vertical" (id 2) (at 48.26 26.67 0)
+      (effects (font (size 1.27 1.27)) hide)
+    )
+    (property "Datasheet" "~" (id 3) (at 48.26 26.67 0)
+      (effects (font (size 1.27 1.27)) hide)
+    )
+    (property "LCSC" "C144395" (id 4) (at 48.26 26.67 0)
       (effects (font (size 1.27 1.27)) hide)
     )
@@
   (symbol (lib_id "Device:R") (at 29.21 58.42 0) (unit 1)
     (in_bom yes) (on_board yes)
-    (property "Reference" "R?" (id 0) (at 30.48 57.15 0)
+    (property "Reference" "R1" (id 0) (at 30.48 57.15 0)
       (effects (font (size 1.27 1.27)) (justify left))
     )
@@
   (symbol (lib_id "Device:C") (at 39.37 68.58 0) (unit 1)
     (in_bom yes) (on_board yes) (fields_autoplaced)
-    (property "Reference" "C?" (id 0) (at 43.18 67.3099 0)
+    (property "Reference" "C1" (id 0) (at 43.18 67.3099 0)
       (effects (font (size 1.27 1.27)) (justify left))
     )
@@
   (symbol (lib_id "Device:R") (at 29.21 68.58 0) (unit 1)
     (in_bom yes) (on_board yes)
-    (property "Reference" "R?" (id 0) (at 30.48 67.31 0)
+    (property "Reference" "R2" (id 0) (at 30.48 67.31 0)
       (effects (font (size 1.27 1.27)) (justify left))
     )
@@
   (symbol (lib_id "power:GND") (at 29.21 74.93 0) (unit 1)
     (in_bom yes) (on_board yes)
-    (property "Reference" "#PWR?" (id 0) (at 29.21 81.28 0)
+    (property "Reference" "#PWR0103" (id 0) (at 29.21 81.28 0)
       (effects (font (size 1.27 1.27)) hide)
     )
@@
   (symbol (lib_id "MeineBibli:+4V5") (at 41.91 58.42 0) (unit 1)
     (in_bom yes) (on_board yes)
-    (property "Reference" "#PWR?" (id 0) (at 41.91 62.23 0)
+    (property "Reference" "#PWR0101" (id 0) (at 41.91 62.23 0)
       (effects (font (size 1.27 1.27)) hide)
     )
@@
       (reference "#PWR04") (unit 1) (value "GND") (footprint "")
     )
+    (path "/c2d81a3b-9b02-4ddc-9c7b-c0e881678970"
+      (reference "#PWR0101") (unit 1) (value "+4V5") (footprint "")
+    )
     (path "/09433d97-62ec-42de-89f2-7d0b68dc1b9d"
-      (reference "#PWR?") (unit 1) (value "GND") (footprint "")
+      (reference "#PWR0102") (unit 1) (value "GND") (footprint "")
+    )
+    (path "/b9272e8b-2d00-4d6b-ae8c-fd62ef331586"
+      (reference "#PWR0103") (unit 1) (value "GND") (footprint "")
     )
     (path "/296b967f-b7a9-453f-856a-7b874fdca3db"
-      (reference "#PWR?") (unit 1) (value "+9V") (footprint "")
-    )
-    (path "/b9272e8b-2d00-4d6b-ae8c-fd62ef331586"
-      (reference "#PWR?") (unit 1) (value "GND") (footprint "")
-    )
-    (path "/c2d81a3b-9b02-4ddc-9c7b-c0e881678970"
-      (reference "#PWR?") (unit 1) (value "+4V5") (footprint "")
+      (reference "#PWR0104") (unit 1) (value "+9V") (footprint "")
+    )
+    (path "/8672a05d-b750-4ddd-a92d-4c58fddcdd4e"
+      (reference "C1") (unit 1) (value "22uF") (footprint "Capacitor_SMD:C_1206_3216Metric")
     )
     (path "/75f89342-e5fb-4ec8-a9a1-4514a000c1c5"
@@
       (reference "C102") (unit 1) (value "220nF") (footprint "Capacitor_SMD:C_0603_1608Metric")
     )
-    (path "/8672a05d-b750-4ddd-a92d-4c58fddcdd4e"
-      (reference "C?") (unit 1) (value "22uF") (footprint "Capacitor_SMD:C_1206_3216Metric")
-    )
     (path "/43624bd7-5b28-4455-bedf-a59e39f0128d"
       (reference "J1") (unit 1) (value "Conn_01x04") (footprint "Connector_JST:JST_XH_B4B-XH-A_1x04_P2.50mm_Vertical")
@@
       (reference "JP100") (unit 1) (value "Jmp") (footprint "Jumper:SolderJumper-2_P1.3mm_Open_TrianglePad1.0x1.5mm")
     )
+    (path "/4e944601-14c5-4478-a9d6-8d2ad19dcc43"
+      (reference "R1") (unit 1) (value "10K") (footprint "Resistor_SMD:R_0603_1608Metric")
+    )
+    (path "/8d9ea4cf-1047-42af-bf72-13258f22d6ad"
+      (reference "R2") (unit 1) (value "10K") (footprint "Resistor_SMD:R_0603_1608Metric")
+    )
     (path "/97468472-fb1b-477a-a19a-eda9fd340e0b"
       (reference "R100") (unit 1) (value "1M") (footprint "Resistor_SMD:R_0603_1608Metric")
@@
       (reference "R103") (unit 1) (value "2k2") (footprint "Resistor_SMD:R_0603_1608Metric")
     )
-    (path "/4e944601-14c5-4478-a9d6-8d2ad19dcc43"
-      (reference "R?") (unit 1) (value "10K") (footprint "Resistor_SMD:R_0603_1608Metric")
-    )
-    (path "/8d9ea4cf-1047-42af-bf72-13258f22d6ad"
-      (reference "R?") (unit 1) (value "10K") (footprint "Resistor_SMD:R_0603_1608Metric")
-    )
     (path "/eade452d-0fd2-478e-ba2c-c8c7cc57b518"

Commit message: [404][UpperRaw] Apply learned lessons from TOP:
- Name on silk etc. is now a text variable
- Optimized copypasta parts
- Set pot footprint to my modified one
- Rename pots ro always be RV1-6
- Use text variables for pot names
- Show pot values on silk
- Update board constraints to JLCPCB capabilities
- Add Gndpour to UpperRaw
- Set "Not in schematic" for OSHW logo
Parts:
- removed C100: 100uF, Capacitor_THT:CP_Radial_D5.0mm_P2.00mm, symbol Device:C_Polarized
- C1: value 22uF -> (none); footprint Capacitor_SMD:C_1206_3216Metric -> (none)
- C101: value 10uF -> (none); footprint Capacitor_SMD:C_0805_2012Metric -> (none)
- C102: value 220nF -> (none); footprint Capacitor_SMD:C_0603_1608Metric -> (none)
- J1: value Conn_01x04 -> (none); footprint Connector_JST:JST_XH_B4B-XH-A_1x04_P2.50mm_Vertical -> (none)
- JP100: value Jmp -> (none); footprint Jumper:SolderJumper-2_P1.3mm_Open_TrianglePad1.0x1.5mm -> (none)
- R1, R2: value 10K -> (none); footprint Resistor_SMD:R_0603_1608Metric -> (none)
- R100: value 1M -> (none); footprint Resistor_SMD:R_0603_1608Metric -> (none)
- R101: value 2M2 -> (none); footprint Resistor_SMD:R_0603_1608Metric -> (none)
- R102: value 390R -> (none); footprint Resistor_SMD:R_0603_1608Metric -> (none)
- R103: value 2k2 -> (none); footprint Resistor_SMD:R_0603_1608Metric -> (none)
- RV1: renamed from RV102; value 100K Lin -> (none); footprint Potentiometer_THT:Potentiometer_Alpha_RD901F-40-00D_Single_Vertical -> (none)
- RV2: renamed from RV101; value 100K Lin -> (none); footprint Potentiometer_THT:Potentiometer_Alpha_RD901F-40-00D_Single_Vertical -> (none)
- RV3: renamed from RV100; value 100K Lin -> (none); footprint Potentiometer_THT:Potentiometer_Alpha_RD901F-40-00D_Single_Vertical -> (none)
- RV4: renamed from RV202; value 100K Lin -> (none); footprint Potentiometer_THT:Potentiometer_Alpha_RD901F-40-00D_Single_Vertical -> (none)
- RV5: renamed from RV201; value 100K Lin -> (none); footprint Potentiometer_THT:Potentiometer_Alpha_RD901F-40-00D_Single_Vertical -> (none)
- RV6: renamed from RV200; value 100K Lin -> (none); footprint Potentiometer_THT:Potentiometer_Alpha_RD901F-40-00D_Single_Vertical -> (none)
- SW100, SW101, SW200, SW201: value SW_DPDT_x2 -> (none); footprint MeineBib:Switch_toggle_DPDT_Print -> (none)
- SW102, SW103, SW202, SW203: value SW_SPDT -> (none); footprint MeineBib:Switch_toggle_SPDT_Print -> (none)
- TP100: value TP -> (none); footprint TestPoint:TestPoint_Pad_D2.0mm -> (none)
Other:
- note added: "${RV1}"
- note added: "${RV2}"
- note added: "${RV3}"
- note added: "${RV4}"
- note added: "${RV5}"
- note added: "${RV6}"
