File: pcb/TOP_Frontpanel/TOP_Frontpanel.kicad_pcb (KiCad board)
At the start: 2 copper layers, 54.5 x 106.4 mm, 19 parts

Commit message: [TOP] Create frontpanel
Parts:
- removed the REF** at (149.4, 95.3)
- removed the REF** at (166.7, 69.6)
- removed the REF** at (166.7, 95.3)
- removed the REF** at (132.2, 95.3)
- removed the REF** at (132.2, 69.6)
- removed the REF** at (149.4, 69.6)
- renumbered REF** to Bass, REF** to Gain, REF** to Mid, REF** to Midrange, REF** to Treble, REF** to Vol
Routing:
- net (no net): track 0.00 -> 384.1 mm, vias 0 -> 11
Other:
- board text added: "TOP"
- board text removed: "Base"
