File: pcb/YOU WHAT?!/YOU WHAT?!.kicad_pcb (KiCad board)
At the start: 2 copper layers, 52 x 63 mm, 34 parts, among them J1 Conn_01x04, SW100 SW_DPDT_x2, SW101 SW_DPDT_x2, SW102 SW_SPDT, SW103 SW_SPDT, SW200 SW_DPDT_x2, SW201 SW_DPDT_x2, SW202 SW_SPDT, SW203 SW_SPDT

Commit message: [YW] Start creating PCB
Parts:
- removed C1: 22uF, Capacitor_SMD:C_1206_3216Metric
- removed C101: 10uF, Capacitor_SMD:C_0805_2012Metric
- removed C102: 220nF, Capacitor_SMD:C_0603_1608Metric
- removed JP100: Jmp, Jumper:SolderJumper-2_P1.3mm_Open_TrianglePad1.0x1.5mm
- removed R101: 2M2, Resistor_SMD:R_0603_1608Metric
- removed R102: 390R, Resistor_SMD:R_0603_1608Metric
- removed R103: 2k2, Resistor_SMD:R_0603_1608Metric
- removed R2: 10K, Resistor_SMD:R_0603_1608Metric
- removed the REF** at (149.5, 116.8)
- removed RV2: 100K Lin, MeineBib:Potentiometer_Alpha_RD901F-40-00D_Single_Vertical
- removed SW100, SW101, SW200, SW201: SW_DPDT_x2, MeineBib:Switch_toggle_DPDT_Print
- removed SW102, SW103, SW202, SW203: SW_SPDT, MeineBib:Switch_toggle_SPDT_Print
- removed TP100: TP, TestPoint:TestPoint_Pad_D2.0mm
- added C10: 1nF, Capacitor_SMD:C_0603_1608Metric, F.Cu at (90.6, 98.6)
- added C11: 220nF, Capacitor_SMD:C_0603_1608Metric, F.Cu at (107.1, 85.1)
- added C12: 1nF, Capacitor_SMD:C_0603_1608Metric, F.Cu at (101.2, 87.6)
- added C13: 22nF, Capacitor_SMD:C_0603_1608Metric, F.Cu at (86.6, 94.4)
- added C14: 1nF, Capacitor_SMD:C_0603_1608Metric, F.Cu at (93.2, 91.1)
- added C15: 22nF, Capacitor_SMD:C_0603_1608Metric, F.Cu at (163.2, 73.2)
- added C16: 10nF, Capacitor_SMD:C_0603_1608Metric, F.Cu at (164.1, 86.0)
- added C17: 47nF, Capacitor_SMD:C_0603_1608Metric, F.Cu at (164.2, 113.6)
- added C18: 47nF, Capacitor_SMD:C_0603_1608Metric, F.Cu at (164.1, 93.2)
- added C19: 10nF, Capacitor_SMD:C_0603_1608Metric, F.Cu at (169.6, 73.2)
- added C2: 100uF, Capacitor_SMD:CP_Elec_6.3x5.3, F.Cu at (156.2, 117.3)
- added C20: 47pF, Capacitor_SMD:C_0603_1608Metric, F.Cu at (143.8, 89.6)
- added C21: 47pF, Capacitor_SMD:C_0603_1608Metric, F.Cu at (143.8, 93.2)
- added C22: 47pF, Capacitor_SMD:C_0603_1608Metric, F.Cu at (155.2, 89.6)
- added C23: 47pF, Capacitor_SMD:C_0603_1608Metric, F.Cu at (155.2, 93.2)
- added C4: 47nF, Capacitor_SMD:C_0603_1608Metric, F.Cu at (170.3, 120.3)
- added C6: 47pF, Capacitor_SMD:C_0603_1608Metric, F.Cu at (168.2, 120.3)
- added C7: 220nF, Capacitor_SMD:C_0603_1608Metric, F.Cu at (95.1, 85.1)
- added C8: 47nF, Capacitor_SMD:C_0603_1608Metric, F.Cu at (107.9, 80.1)
- added C9: 47nF, Capacitor_SMD:C_0603_1608Metric, F.Cu at (99.9, 80.1)
- added Q1: BC849C, Package_TO_SOT_SMD:SOT-23, F.Cu at (167.5, 116.0)
- added R11: 10k, Resistor_SMD:R_0603_1608Metric, F.Cu at (98.6, 92.7)
- added R12: 27k, Resistor_SMD:R_0603_1608Metric, F.Cu at (103.9, 82.6)
- added R13: 1M, Resistor_SMD:R_0603_1608Metric, F.Cu at (90.6, 96.1)
- added R14: 10k, Resistor_SMD:R_0603_1608Metric, F.Cu at (162.1, 86.0)
- added R15: 27k, Resistor_SMD:R_0603_1608Metric, F.Cu at (161.2, 73.2)
- added R16: 10M, Resistor_SMD:R_0603_1608Metric, F.Cu at (165.2, 73.2)
- added R17: 27k, Resistor_SMD:R_0603_1608Metric, F.Cu at (162.1, 93.2)
- added R18: 220k, Resistor_SMD:R_0603_1608Metric, F.Cu at (162.1, 89.6)
- added R19: 47k, Resistor_SMD:R_0603_1608Metric, F.Cu at (162.2, 113.6)
- added R20: 1k, Resistor_SMD:R_0603_1608Metric, F.Cu at (164.1, 89.6)
- added R21: 10k, Resistor_SMD:R_0603_1608Metric, F.Cu at (167.5, 73.2)
- added R3: 10k, Resistor_SMD:R_0603_1608Metric, F.Cu at (107.9, 82.6)
- added R4: 4k7, Resistor_SMD:R_0603_1608Metric, F.Cu at (162.1, 120.3)
- added R6: 220k, Resistor_SMD:R_0603_1608Metric, F.Cu at (94.6, 98.6)
- added R7: 10k, Resistor_SMD:R_0603_1608Metric, F.Cu at (86.6, 96.9)
- added R8: 27k, Resistor_SMD:R_0603_1608Metric, F.Cu at (94.6, 93.6)
- added R9: 10k, Resistor_SMD:R_0603_1608Metric, F.Cu at (98.6, 95.2)
- added TP1: PostInp, TestPoint:TestPoint_Pad_D2.0mm, F.Cu at (172.1, 116.0)
- added TP2: 9V, TestPoint:TestPoint_Pad_D2.0mm, F.Cu at (145.4, 120.1)
- added TP3: 4V5, TestPoint:TestPoint_Pad_D2.0mm, F.Cu at (150.8, 120.1)
- added TP4: PostGain, TestPoint:TestPoint_Pad_D2.0mm, F.Cu at (173.1, 81.7)
- added TP5: PostTone, TestPoint:TestPoint_Pad_D2.0mm, F.Cu at (132.4, 107.4)
- added U1: HEF4069UB, Package_SO:SOIC-14_3.9x8.7mm_P1.27mm, F.Cu at (149.5, 90.0)
- R1: value 10K -> 10k
- RV1, RV3: value 100K Lin -> 500K Lin
- RV4: value 100K Lin -> 500K Log
- RV5: value 100K Lin -> 10K Lin
- moved R1 100.6 mm to (166.2, 120.3), turned to 90 degrees
- moved R22 80.8 mm to (164.2, 120.3), turned to 90 degrees
- renumbered R100 to R22
Connections:
- R1 pad 1: +9V -> Upper_PCB_Input
- R1 pad 2: +4V5 -> Net-(C4-Pad1)
- R22 pad 1: unconnected-(R100-Pad1) -> +4V5
- R22 pad 2: unconnected-(R100-Pad2) -> Net-(C4-Pad2)
- RV1 pad 1: unconnected-(RV1-Pad1) -> Net-(C15-Pad1)
- RV1 pad 2: unconnected-(RV1-Pad2) -> Net-(C22-Pad2)
- RV1 pad 3: unconnected-(RV1-Pad3) -> Net-(C19-Pad1)
- RV3 pad 1: unconnected-(RV3-Pad1) -> Net-(C21-Pad1)
- RV3 pad 2: unconnected-(RV3-Pad2) -> Net-(R7-Pad2)
- RV3 pad 3: unconnected-(RV3-Pad3) -> Net-(R7-Pad2)
- RV4 pad 1: unconnected-(RV4-Pad1) -> Net-(RV4-Pad1)
- RV4 pad 2: unconnected-(RV4-Pad2) -> Net-(C9-Pad2)
- RV4 pad 3: unconnected-(RV4-Pad3) -> Net-(C9-Pad2)
- RV5 pad 1: unconnected-(RV5-Pad1) -> GND
- RV5 pad 2: unconnected-(RV5-Pad2) -> Net-(C8-Pad2)
- RV5 pad 3: unconnected-(RV5-Pad3) -> Net-(RV4-Pad1)
- RV6 pad 1: unconnected-(RV6-Pad1) -> Net-(C9-Pad2)
- RV6 pad 2: unconnected-(RV6-Pad2) -> Net-(C7-Pad1)
- RV6 pad 3: unconnected-(RV6-Pad3) -> Net-(C10-Pad2)
Routing:
- net Net-(C20-Pad1): track 0.00 -> 37.4 mm, vias 0 -> 2
- net Net-(C23-Pad1): track 0.00 -> 37.2 mm
- net +9V: track 0.00 -> 34.5 mm
- net Net-(C22-Pad2): track 0.00 -> 32.7 mm, vias 0 -> 2
- net Net-(C22-Pad1): track 0.00 -> 30.8 mm
- net Net-(C16-Pad1): track 0.00 -> 23.3 mm, vias 0 -> 2
- net +4V5: track 0.00 -> 20.0 mm
- net Upper_PCB_Input: track 0.00 -> 15.8 mm
- net Net-(C19-Pad1): track 0.00 -> 15.0 mm
- net Net-(C4-Pad2): track 0.00 -> 9.66 mm
- net Net-(C17-Pad1): track 0.00 -> 8.55 mm
- net Net-(C4-Pad1): track 0.00 -> 5.16 mm
- net Net-(C15-Pad2): track 0.00 -> 4.75 mm
- net Net-(R17-Pad1): track 0.00 -> 4.62 mm
- net Net-(C11-Pad1): track 0.00 -> 3.82 mm
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Other:
- board text removed: "Either delete mounting hole or pot"

Commit message: [YW] Finish initial version of PCB
Parts:
- moved C9 72.0 mm to (166.8, 106.9), turned to -90 degrees
- moved R3 66.1 mm to (166.3, 113.6), turned to 90 degrees
- moved R7 55.3 mm to (141.8, 93.0), turned to -90 degrees
- moved R13 51.6 mm to (141.8, 89.6), turned to -90 degrees
- moved C8 49.4 mm to (149.5, 106.9), turned to -90 degrees
- moved C13 47.2 mm to (133.5, 89.6), turned to 90 degrees
- moved C14 44.5 mm to (137.7, 89.6), turned to -90 degrees
- moved C7 43.2 mm to (132.4, 106.9), turned to 90 degrees
- moved C10 41.2 mm to (131.3, 93.0), turned to -90 degrees
- moved R6 39.3 mm to (133.5, 93.0), turned to -90 degrees
- moved R9 39.2 mm to (137.7, 93.0), turned to -90 degrees
- moved R11 37.2 mm to (135.7, 89.6), turned to -90 degrees
- moved R8 37.0 mm to (131.3, 89.6), turned to 90 degrees
- moved R12 36.5 mm to (139.7, 89.6), turned to -90 degrees
- moved C12 34.9 mm to (135.7, 93.0), turned to 90 degrees
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Routing:
- net Net-(C8-Pad1): track 0.00 -> 54.7 mm, vias 0 -> 2
- net Upper_PCB_Output: track 0.00 -> 44.4 mm, vias 0 -> 3
- net +4V5: track 20.0 -> 60.0 mm, vias 0 -> 2
- net Net-(C21-Pad1): track 3.71 -> 42.8 mm, vias 0 -> 3
- net Net-(C9-Pad2): track 2.50 -> 37.7 mm, vias 0 -> 2
- net Net-(R7-Pad2): track 2.50 -> 33.9 mm, vias 0 -> 2
- net Net-(C15-Pad2): track 4.75 -> 30.0 mm, vias 0 -> 2
- net Net-(RV4-Pad1): track 0.00 -> 24.1 mm
- net Net-(C22-Pad1): track 30.8 -> 11.2 mm, vias 0 -> 2
- net Net-(C10-Pad2): track 0.00 -> 17.6 mm
- net Net-(C20-Pad1): track 37.4 -> 23.2 mm
- net Net-(C16-Pad1): track 23.3 -> 10.1 mm, vias 2 -> 0
- net Net-(C7-Pad2): track 0.00 -> 12.7 mm
- net Net-(C10-Pad1): track 0.00 -> 12.5 mm
- net Net-(C19-Pad2): track 2.69 -> 13.4 mm
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Other:
- board text added: "YOU WHAT?!"
- board text removed: "${RV2}"
