File: pcb/YOU WHAT/YOU WHAT.kicad_pcb (KiCad board)
At the start: 2 copper layers, 52 x 63 mm, 59 parts, among them J1 Conn_01x04, Q1 BC849C, U1 HEF4069UB

Commit message: [YW] Rename project; Fix R6/R18 BOM
Changed lines of the file:
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@@
       (layerselection 0x00010fc_ffffffff)
       (disableapertmacros false)
-      (usegerberextensions false)
-      (usegerberattributes true)
-      (usegerberadvancedattributes true)
-      (creategerberjobfile true)
+      (usegerberextensions true)
+      (usegerberattributes false)
+      (usegerberadvancedattributes false)
+      (creategerberjobfile false)
       (svguseinch false)
       (svgprecision 6)
@@
       (plotinvisibletext false)
       (sketchpadsonfab false)
-      (subtractmaskfromsilk false)
+      (subtractmaskfromsilk true)
       (outputformat 1)
       (mirror false)
-      (drillshape 1)
+      (drillshape 0)
       (scaleselection 1)
-      (outputdirectory "")
-    )
-  )
-  (property "Commit" "Commit")
+      (outputdirectory "production_files/")
+    )
+  )
+  (property "Commit" "d8db029")
   (property "Link" "gitlab.com/Chrismettal/pedaldev")
   (property "Name" "YOU WHAT?!")
@@
     (fp_line (start 0 -1.35) (end 0.625 -2.35) (layer "F.Fab") (width 0.1))
     (fp_line (start -2.45 3.4) (end 9.95 3.4) (layer "F.Fab") (width 0.1))
-    (pad "1" thru_hole roundrect (at 0 0 180) (size 1.7 1.95) (drill 0.95) (layers *.Cu *.Mask) (roundrect_rratio 0.147059)
+    (pad "1" thru_hole roundrect (at 0 0 180) (size 1.7 1.95) (drill 0.95) (layers *.Cu *.Mask) (roundrect_rratio 0.1470588235)
       (net 3 "Upper_PCB_Input") (pinfunction "Pin_1") (pintype "passive"))
     (pad "2" thru_hole oval (at 2.5 0 180) (size 1.7 1.95) (drill 0.95) (layers *.Cu *.Mask)
