File: pcb/YOU WHAT/YOU WHAT.kicad_sch (KiCad schematic)
At the start: 52 parts, among them J1 Conn_01x04, Q1 BC849C, U1 HEF4069UB

Commit message: [YW] Rename project; Fix R6/R18 BOM
Parts:
- R18, R6: LCSC C17556 -> C22961
Changed lines of the file:
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@@
       (effects (font (size 1.27 1.27)) hide)
     )
-    (property "LCSC" "C17556" (id 4) (at 295.91 109.22 0)
+    (property "LCSC" "C22961" (id 4) (at 295.91 109.22 0)
       (effects (font (size 1.27 1.27)) hide)
     )
@@
       (effects (font (size 1.27 1.27)) hide)
     )
-    (property "LCSC" "C17556" (id 4) (at 113.03 170.18 0)
-      (effects (font (size 1.27 1.27)) hide)
-    )
+    (property "LCSC" "C22961" (id 4) (at 113.03 170.18 0)
+      (effects (font (size 1.27 1.27)) hide)
+    )
