File: pcb/YOU WHAT_Frontpanel/YOU WHAT_Frontpanel.kicad_pcb (KiCad board)
At the start: 2 copper layers, 54.5 x 106.4 mm, 13 parts

Commit message: [YW] Finish initial frontpanel design
Routing:
- net (no net): track 0.00 -> 120.7 mm
Changed lines of the file:
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@@
     (effects (font (size 8 8) (thickness 1.2)))
   )
+  (segment (start 129.638 133.907) (end 124.304 128.573) (width 0.4) (layer "F.Cu") (net 0))
+  (segment (start 160.626 142.162) (end 166.976 135.812) (width 0.4) (layer "F.Cu") (net 0))
+  (segment (start 167.0395 136.5105) (end 167.23 136.32) (width 0.4) (layer "F.Cu") (net 0))
+  (segment (start 174.723 128.827) (end 169.77 133.78) (width 0.4) (layer "F.Cu") (net 0))
+  (segment (start 160.88 142.67) (end 167.0395 136.5105) (width 0.4) (layer "F.Cu") (net 0))
+  (segment (start 129.7015 134.7325) (end 124.177 129.208) (width 0.4) (layer "F.Cu") (net 0))
+  (segment (start 140.052 154.227) (end 137.893 154.227) (width 0.4) (layer "F.Cu") (net 0))
+  (segment (start 158.848 154.227) (end 160.88 154.227) (width 0.4) (layer "F.Cu") (net 0))
+  (segment (start 137.639 142.67) (end 133.2575 138.2885) (width 0.4) (layer "F.Cu") (net 0))
+  (segment (start 156.308 142.162) (end 160.626 142.162) (width 0.4) (layer "F.Cu") (net 0))
+  (segment (start 164.309 156.894) (end 164.436 157.021) (width 0.4) (layer "F.Cu") (net 0))
+  (segment (start 160.88 154.227) (end 163.674 157.021) (width 0.4) (layer "F.Cu") (net 0))
+  (segment (start 137.893 142.162) (end 137.004 141.273) (width 0.4) (layer "F.Cu") (net 0))
+  (segment (start 128.749 162.609) (end 128.495 162.863) (width 0.4) (layer "F.Cu") (net 0))
+  (segment (start 140.179 153.719) (end 137.639 153.719) (width 0.4) (layer "F.Cu") (net 0))
+  (segment (start 137.893 154.227) (end 129.257 162.863) (width 0.4) (layer "F.Cu") (net 0))
+  (segment (start 142.211 142.67) (end 137.639 142.67) (width 0.4) (layer "F.Cu") (net 0))
+  (segment (start 156.816 142.67) (end 160.88 142.67) (width 0.4) (layer "F.Cu") (net 0))
+  (segment (start 142.719 142.162) (end 137.893 142.162) (width 0.4) (layer "F.Cu") (net 0))
+  (segment (start 174.723 128.065) (end 169.77 133.018) (width 0.4) (layer "F.Cu") (net 0))
+  (segment (start 137.004 141.273) (end 135.48 139.749) (width 0.4) (layer "F.Cu") (net 0))
+  (segment (start 137.893 142.162) (end 135.48 139.749) (width 0.4) (layer "F.Cu") (net 0))
+  (segment (start 137.639 153.719) (end 128.749 162.609) (width 0.4) (layer "F.Cu") (net 0))
+  (segment (start 159.102 153.719) (end 161.134 153.719) (width 0.4) (layer "F.Cu") (net 0))
+  (segment (start 161.134 153.719) (end 164.309 156.894) (width 0.4) (layer "F.Cu") (net 0))
   (zone (net 0) (net_name "") (layers F&B.Cu) (hatch edge 0.508)
     (connect_pads (clearance 0.508))
